Commit message: agggg not working

File: robota.urdf (robot description, URDF)
Before this commit: robot robot, 3 links, 2 joints
Joints:
- joint Torso_BackLeg: origin xyz=-6.5 2 1 rpy=0 0 0 -> xyz=0.5 5 1 rpy=0 0 0
- joint Torso_FrontLeg: origin xyz=-5.5 2 1 rpy=0 0 0 -> xyz=1.5 5 1 rpy=0 0 0

File: robotb.urdf (robot description, URDF)
Before this commit: robot robot, 3 links, 2 joints
Joints:
- joint Torso_BackLeg: axis 1 0 0 -> 0 1 0; origin xyz=-0.5 0 1 rpy=0 0 0 -> xyz=7.5 4 1 rpy=0 0 0
- joint Torso_FrontLeg: axis 1 0 0 -> 0 1 0; origin xyz=0.5 0 1 rpy=0 0 0 -> xyz=8.5 4 1 rpy=0 0 0
