Commit message: have two robots in the world, run from test

File: robot_A.urdf (robot description, URDF)
Before this commit: robot robot, 1 links, 0 joints
Links:
- removed link Torso_A
- added link BackLeg, mass 1; collision box size=1 1 1; visual box size=1 1 1
- added link FrontLeg, mass 1; collision box size=1 1 1; visual box size=1 1 1
- added link Torso, mass 1; collision box size=1 1 1; visual box size=1 1 1
Joints:
- added joint Torso_BackLeg: type revolute, parent Torso, child BackLeg, origin xyz=6.5 -2 1 rpy=0 0 0, axis 0 1 0, limit lower=-3.14159 upper=3.14159 effort=0.0 velocity=0.0
- added joint Torso_FrontLeg: type revolute, parent Torso, child FrontLeg, origin xyz=7.5 -2 1 rpy=0 0 0, axis 0 1 0, limit lower=-3.14159 upper=3.14159 effort=0.0 velocity=0.0

File: robot_B.urdf (robot description, URDF)
Before this commit: robot robot, 1 links, 0 joints
Links:
- removed link Torso_B
- added link BackLeg, mass 1; collision box size=1 1 1; visual box size=1 1 1
- added link FrontLeg, mass 1; collision box size=1 1 1; visual box size=1 1 1
- added link Torso, mass 1; collision box size=1 1 1; visual box size=1 1 1
Joints:
- added joint Torso_BackLeg: type revolute, parent Torso, child BackLeg, origin xyz=4.5 7 1 rpy=0 0 0, axis 0 1 0, limit lower=-3.14159 upper=3.14159 effort=0.0 velocity=0.0
- added joint Torso_FrontLeg: type revolute, parent Torso, child FrontLeg, origin xyz=5.5 7 1 rpy=0 0 0, axis 0 1 0, limit lower=-3.14159 upper=3.14159 effort=0.0 velocity=0.0

Commit message: robots move, they just have the same synapse weights

File: robot_A.urdf (robot description, URDF)
Before this commit: robot robot, 3 links, 2 joints
Joints:
- joint Torso_BackLeg: origin xyz=6.5 -2 1 rpy=0 0 0 -> xyz=-10.5 -5 1 rpy=0 0 0
- joint Torso_FrontLeg: origin xyz=7.5 -2 1 rpy=0 0 0 -> xyz=-9.5 -5 1 rpy=0 0 0

File: robot_B.urdf (robot description, URDF)
Before this commit: robot robot, 3 links, 2 joints
Joints:
- joint Torso_BackLeg: origin xyz=4.5 7 1 rpy=0 0 0 -> xyz=-2.5 -5 1 rpy=0 0 0
- joint Torso_FrontLeg: origin xyz=5.5 7 1 rpy=0 0 0 -> xyz=-1.5 -5 1 rpy=0 0 0

Commit message: milestone 1!

File: robot_A.urdf (robot description, URDF)
Before this commit: robot robot, 3 links, 2 joints
Joints:
- joint Torso_BackLeg: origin xyz=-10.5 -5 1 rpy=0 0 0 -> xyz=7.5 -1 1 rpy=0 0 0
- joint Torso_FrontLeg: origin xyz=-9.5 -5 1 rpy=0 0 0 -> xyz=8.5 -1 1 rpy=0 0 0

File: robot_B.urdf (robot description, URDF)
Before this commit: robot robot, 3 links, 2 joints
Joints:
- joint Torso_BackLeg: origin xyz=-2.5 -5 1 rpy=0 0 0 -> xyz=1.5 -4 1 rpy=0 0 0
- joint Torso_FrontLeg: origin xyz=-1.5 -5 1 rpy=0 0 0 -> xyz=2.5 -4 1 rpy=0 0 0

Commit message: why aren't they walking

File: robot_A.urdf (robot description, URDF)
Before this commit: robot robot, 3 links, 2 joints
Joints:
- joint Torso_BackLeg: origin xyz=-7.5 9 1 rpy=0 0 0 -> xyz=-4.5 1 1 rpy=0 0 0
- joint Torso_FrontLeg: origin xyz=-6.5 9 1 rpy=0 0 0 -> xyz=-3.5 1 1 rpy=0 0 0

File: robot_B.urdf (robot description, URDF)
Before this commit: robot robot, 3 links, 2 joints
Joints:
- joint Torso_BackLeg: origin xyz=-2.5 -3 1 rpy=0 0 0 -> xyz=-7.5 -10 1 rpy=0 0 0
- joint Torso_FrontLeg: origin xyz=-1.5 -3 1 rpy=0 0 0 -> xyz=-6.5 -10 1 rpy=0 0 0

Commit message: robot changes

File: robot_A.urdf (robot description, URDF)
Before this commit: robot robot, 3 links, 2 joints
Joints:
- joint Torso_BackLeg: origin xyz=-4.5 1 1 rpy=0 0 0 -> xyz=-1.5 10 1 rpy=0 0 0
- joint Torso_FrontLeg: origin xyz=-3.5 1 1 rpy=0 0 0 -> xyz=-0.5 10 1 rpy=0 0 0

File: robot_B.urdf (robot description, URDF)
Before this commit: robot robot, 3 links, 2 joints
Joints:
- joint Torso_BackLeg: origin xyz=-7.5 -10 1 rpy=0 0 0 -> xyz=-5.5 -8 1 rpy=0 0 0
- joint Torso_FrontLeg: origin xyz=-6.5 -10 1 rpy=0 0 0 -> xyz=-4.5 -8 1 rpy=0 0 0

Commit message: working again after head reset?

File: robot_A.urdf (robot description, URDF)
Before this commit: robot robot, 3 links, 2 joints
Joints:
- joint Torso_BackLeg: origin xyz=7.5 -1 1 rpy=0 0 0 -> xyz=-3.5 -2 1 rpy=0 0 0
- joint Torso_FrontLeg: origin xyz=8.5 -1 1 rpy=0 0 0 -> xyz=-2.5 -2 1 rpy=0 0 0

File: robot_B.urdf (robot description, URDF)
Before this commit: robot robot, 3 links, 2 joints
Joints:
- joint Torso_BackLeg: origin xyz=1.5 -4 1 rpy=0 0 0 -> xyz=-4.5 -8 1 rpy=0 0 0
- joint Torso_FrontLeg: origin xyz=2.5 -4 1 rpy=0 0 0 -> xyz=-3.5 -8 1 rpy=0 0 0

Commit message: why aren't they walking???????????

File: robot_A.urdf (robot description, URDF)
Before this commit: robot robot, 3 links, 2 joints
Joints:
- joint Torso_BackLeg: origin xyz=-3.5 -2 1 rpy=0 0 0 -> xyz=7.5 10 1 rpy=0 0 0
- joint Torso_FrontLeg: origin xyz=-2.5 -2 1 rpy=0 0 0 -> xyz=8.5 10 1 rpy=0 0 0

Commit message: amazing they walk now and all is good

File: robot_A.urdf (robot description, URDF)
Before this commit: robot robot, 3 links, 2 joints
Joints:
- joint Torso_BackLeg: origin xyz=7.5 10 1 rpy=0 0 0 -> xyz=7.5 6 1 rpy=0 0 0
- joint Torso_FrontLeg: origin xyz=8.5 10 1 rpy=0 0 0 -> xyz=8.5 6 1 rpy=0 0 0

File: robot_B.urdf (robot description, URDF)
Before this commit: robot robot, 3 links, 2 joints
Joints:
- joint Torso_BackLeg: origin xyz=-10.5 4 1 rpy=0 0 0 -> xyz=2.5 -9 1 rpy=0 0 0
- joint Torso_FrontLeg: origin xyz=-9.5 4 1 rpy=0 0 0 -> xyz=3.5 -9 1 rpy=0 0 0

Commit message: delete old brains!

File: robot_A.urdf (robot description, URDF)
Before this commit: robot robot, 3 links, 2 joints
Joints:
- joint Torso_BackLeg: origin xyz=7.5 6 1 rpy=0 0 0 -> xyz=-10.5 -5 1 rpy=0 0 0
- joint Torso_FrontLeg: origin xyz=8.5 6 1 rpy=0 0 0 -> xyz=-9.5 -5 1 rpy=0 0 0

File: robot_B.urdf (robot description, URDF)
Before this commit: robot robot, 3 links, 2 joints
Joints:
- joint Torso_BackLeg: origin xyz=2.5 -9 1 rpy=0 0 0 -> xyz=1.5 -10 1 rpy=0 0 0
- joint Torso_FrontLeg: origin xyz=3.5 -9 1 rpy=0 0 0 -> xyz=2.5 -10 1 rpy=0 0 0

Commit message: okay now they seem to have different brains, I don't know that is happening

File: robot_A.urdf (robot description, URDF)
Before this commit: robot robot, 3 links, 2 joints
Joints:
- joint Torso_BackLeg: origin xyz=-10.5 -5 1 rpy=0 0 0 -> xyz=8.5 -10 1 rpy=0 0 0
- joint Torso_FrontLeg: origin xyz=-9.5 -5 1 rpy=0 0 0 -> xyz=9.5 -10 1 rpy=0 0 0

File: robot_B.urdf (robot description, URDF)
Before this commit: robot robot, 3 links, 2 joints
Joints:
- joint Torso_BackLeg: origin xyz=1.5 -10 1 rpy=0 0 0 -> xyz=-2.5 2 1 rpy=0 0 0
- joint Torso_FrontLeg: origin xyz=2.5 -10 1 rpy=0 0 0 -> xyz=-1.5 2 1 rpy=0 0 0

Commit message: okay that time they moved in a different way...

File: robot_A.urdf (robot description, URDF)
Before this commit: robot robot, 3 links, 2 joints
Joints:
- joint Torso_BackLeg: origin xyz=8.5 -10 1 rpy=0 0 0 -> xyz=8.5 -8 1 rpy=0 0 0
- joint Torso_FrontLeg: origin xyz=9.5 -10 1 rpy=0 0 0 -> xyz=9.5 -8 1 rpy=0 0 0

File: robot_B.urdf (robot description, URDF)
Before this commit: robot robot, 3 links, 2 joints
Joints:
- joint Torso_BackLeg: origin xyz=-2.5 2 1 rpy=0 0 0 -> xyz=-0.5 -10 1 rpy=0 0 0
- joint Torso_FrontLeg: origin xyz=-1.5 2 1 rpy=0 0 0 -> xyz=0.5 -10 1 rpy=0 0 0

Commit message: we have some funky stuff going on

File: robot_A.urdf (robot description, URDF)
Before this commit: robot robot, 3 links, 2 joints
Joints:
- joint Torso_BackLeg: origin xyz=8.5 -8 1 rpy=0 0 0 -> xyz=-5.5 -5 1 rpy=0 0 0
- joint Torso_FrontLeg: origin xyz=9.5 -8 1 rpy=0 0 0 -> xyz=-4.5 -5 1 rpy=0 0 0

File: robot_B.urdf (robot description, URDF)
Before this commit: robot robot, 3 links, 2 joints
Joints:
- joint Torso_BackLeg: origin xyz=-0.5 -10 1 rpy=0 0 0 -> xyz=5.5 0 1 rpy=0 0 0
- joint Torso_FrontLeg: origin xyz=0.5 -10 1 rpy=0 0 0 -> xyz=6.5 0 1 rpy=0 0 0

Commit message: vector in space of the position of the robots prints!

File: robot_A.urdf (robot description, URDF)
Before this commit: robot robot, 3 links, 2 joints
Joints:
- joint Torso_BackLeg: origin xyz=-5.5 -5 1 rpy=0 0 0 -> xyz=-2.5 4 1 rpy=0 0 0
- joint Torso_FrontLeg: origin xyz=-4.5 -5 1 rpy=0 0 0 -> xyz=-1.5 4 1 rpy=0 0 0

File: robot_B.urdf (robot description, URDF)
Before this commit: robot robot, 3 links, 2 joints
Joints:
- joint Torso_BackLeg: origin xyz=5.5 0 1 rpy=0 0 0 -> xyz=0.5 -8 1 rpy=0 0 0
- joint Torso_FrontLeg: origin xyz=6.5 0 1 rpy=0 0 0 -> xyz=1.5 -8 1 rpy=0 0 0

Commit message: polar coordinates working all is good

File: robot_A.urdf (robot description, URDF)
Before this commit: robot robot, 3 links, 2 joints
Joints:
- joint Torso_BackLeg: origin xyz=-2.5 4 1 rpy=0 0 0 -> xyz=4.5 -10 1 rpy=0 0 0
- joint Torso_FrontLeg: origin xyz=-1.5 4 1 rpy=0 0 0 -> xyz=5.5 -10 1 rpy=0 0 0

File: robot_B.urdf (robot description, URDF)
Before this commit: robot robot, 3 links, 2 joints
Joints:
- joint Torso_BackLeg: origin xyz=0.5 -8 1 rpy=0 0 0 -> xyz=4.5 4 1 rpy=0 0 0
- joint Torso_FrontLeg: origin xyz=1.5 -8 1 rpy=0 0 0 -> xyz=5.5 4 1 rpy=0 0 0

Commit message: doing stuff in simulation

File: robot_A.urdf (robot description, URDF)
Before this commit: robot robot, 3 links, 2 joints
Joints:
- joint Torso_BackLeg: origin xyz=4.5 -10 1 rpy=0 0 0 -> xyz=7.5 -1 1 rpy=0 0 0
- joint Torso_FrontLeg: origin xyz=5.5 -10 1 rpy=0 0 0 -> xyz=8.5 -1 1 rpy=0 0 0

File: robot_B.urdf (robot description, URDF)
Before this commit: robot robot, 3 links, 2 joints
Joints:
- joint Torso_BackLeg: origin xyz=4.5 4 1 rpy=0 0 0 -> xyz=5.5 5 1 rpy=0 0 0
- joint Torso_FrontLeg: origin xyz=5.5 4 1 rpy=0 0 0 -> xyz=6.5 5 1 rpy=0 0 0

Commit message: trying to make fitness function reward for a smaller r value distance in the polar coordinates between the robots

File: robot_A.urdf (robot description, URDF)
Before this commit: robot robot, 3 links, 2 joints
Joints:
- joint Torso_BackLeg: origin xyz=7.5 -1 1 rpy=0 0 0 -> xyz=2.5 6 1 rpy=0 0 0
- joint Torso_FrontLeg: origin xyz=8.5 -1 1 rpy=0 0 0 -> xyz=3.5 6 1 rpy=0 0 0

File: robot_B.urdf (robot description, URDF)
Before this commit: robot robot, 3 links, 2 joints
Joints:
- joint Torso_BackLeg: origin xyz=5.5 5 1 rpy=0 0 0 -> xyz=-4.5 3 1 rpy=0 0 0
- joint Torso_FrontLeg: origin xyz=6.5 5 1 rpy=0 0 0 -> xyz=-3.5 3 1 rpy=0 0 0

Commit message: put hat on robot

File: robot_A.urdf (robot description, URDF)
Before this commit: robot robot, 3 links, 2 joints
Links:
- added link Hat, mass 1; collision box size=0.25 0.25 0.25; visual box size=0.25 0.25 0.25
Joints:
- added joint Torso_Hat: type revolute, parent Torso, child Hat, origin xyz=9 10 2 rpy=0 0 0, axis 0 1 0, limit lower=-3.14159 upper=3.14159 effort=0.0 velocity=0.0
- joint Torso_BackLeg: origin xyz=2.5 6 1 rpy=0 0 0 -> xyz=8.5 10 1 rpy=0 0 0
- joint Torso_FrontLeg: origin xyz=3.5 6 1 rpy=0 0 0 -> xyz=9.5 10 1 rpy=0 0 0

File: robot_B.urdf (robot description, URDF)
Before this commit: robot robot, 3 links, 2 joints
Links:
- added link Hat, mass 1; collision box size=0.25 0.25 0.25; visual box size=0.25 0.25 0.25
Joints:
- added joint Torso_Hat: type revolute, parent Torso, child Hat, origin xyz=-10 -8 2 rpy=0 0 0, axis 0 1 0, limit lower=-3.14159 upper=3.14159 effort=0.0 velocity=0.0
- joint Torso_BackLeg: origin xyz=-4.5 3 1 rpy=0 0 0 -> xyz=-10.5 -8 1 rpy=0 0 0
- joint Torso_FrontLeg: origin xyz=-3.5 3 1 rpy=0 0 0 -> xyz=-9.5 -8 1 rpy=0 0 0

Commit message: not really working, going to look back at the phc module

File: robot_A.urdf (robot description, URDF)
Before this commit: robot robot, 4 links, 3 joints
Joints:
- joint Torso_BackLeg: origin xyz=8.5 10 1 rpy=0 0 0 -> xyz=-2.5 -1 1 rpy=0 0 0
- joint Torso_FrontLeg: origin xyz=9.5 10 1 rpy=0 0 0 -> xyz=-1.5 -1 1 rpy=0 0 0
- joint Torso_Hat: origin xyz=9 10 2 rpy=0 0 0 -> xyz=-2 -1 2 rpy=0 0 0

File: robot_B.urdf (robot description, URDF)
Before this commit: robot robot, 4 links, 3 joints
Joints:
- joint Torso_BackLeg: origin xyz=-10.5 -8 1 rpy=0 0 0 -> xyz=7.5 -1 1 rpy=0 0 0
- joint Torso_FrontLeg: origin xyz=-9.5 -8 1 rpy=0 0 0 -> xyz=8.5 -1 1 rpy=0 0 0
- joint Torso_Hat: origin xyz=-10 -8 2 rpy=0 0 0 -> xyz=8 -1 2 rpy=0 0 0

Commit message: why do they just stop moving sometimes??

File: robot_A.urdf (robot description, URDF)
Before this commit: robot robot, 4 links, 3 joints
Joints:
- joint Torso_BackLeg: origin xyz=-2.5 -1 1 rpy=0 0 0 -> xyz=-3.5 10 1 rpy=0 0 0
- joint Torso_FrontLeg: origin xyz=-1.5 -1 1 rpy=0 0 0 -> xyz=-2.5 10 1 rpy=0 0 0
- joint Torso_Hat: origin xyz=-2 -1 2 rpy=0 0 0 -> xyz=-3 10 2 rpy=0 0 0

File: robot_B.urdf (robot description, URDF)
Before this commit: robot robot, 4 links, 3 joints
Joints:
- joint Torso_BackLeg: origin xyz=7.5 -1 1 rpy=0 0 0 -> xyz=9.5 10 1 rpy=0 0 0
- joint Torso_FrontLeg: origin xyz=8.5 -1 1 rpy=0 0 0 -> xyz=10.5 10 1 rpy=0 0 0
- joint Torso_Hat: origin xyz=8 -1 2 rpy=0 0 0 -> xyz=10 10 2 rpy=0 0 0

Commit message: ran again

File: robot_A.urdf (robot description, URDF)
Before this commit: robot robot, 4 links, 3 joints
Joints:
- joint Torso_BackLeg: origin xyz=-3.5 10 1 rpy=0 0 0 -> xyz=8.5 5 1 rpy=0 0 0
- joint Torso_FrontLeg: origin xyz=-2.5 10 1 rpy=0 0 0 -> xyz=9.5 5 1 rpy=0 0 0
- joint Torso_Hat: origin xyz=-3 10 2 rpy=0 0 0 -> xyz=9 5 2 rpy=0 0 0

File: robot_B.urdf (robot description, URDF)
Before this commit: robot robot, 4 links, 3 joints
Joints:
- joint Torso_BackLeg: origin xyz=9.5 10 1 rpy=0 0 0 -> xyz=-0.5 5 1 rpy=0 0 0
- joint Torso_FrontLeg: origin xyz=10.5 10 1 rpy=0 0 0 -> xyz=0.5 5 1 rpy=0 0 0
- joint Torso_Hat: origin xyz=10 10 2 rpy=0 0 0 -> xyz=0 5 2 rpy=0 0 0

Commit message: walk but chase sometimes?

File: robot_A.urdf (robot description, URDF)
Before this commit: robot robot, 4 links, 3 joints
Joints:
- joint Torso_BackLeg: origin xyz=8.5 5 1 rpy=0 0 0 -> xyz=-1.5 -1 1 rpy=0 0 0
- joint Torso_FrontLeg: origin xyz=9.5 5 1 rpy=0 0 0 -> xyz=-0.5 -1 1 rpy=0 0 0
- joint Torso_Hat: origin xyz=9 5 2 rpy=0 0 0 -> xyz=-1 -1 2 rpy=0 0 0

File: robot_B.urdf (robot description, URDF)
Before this commit: robot robot, 4 links, 3 joints
Joints:
- joint Torso_BackLeg: origin xyz=-0.5 5 1 rpy=0 0 0 -> xyz=-9.5 -1 1 rpy=0 0 0
- joint Torso_FrontLeg: origin xyz=0.5 5 1 rpy=0 0 0 -> xyz=-8.5 -1 1 rpy=0 0 0
- joint Torso_Hat: origin xyz=0 5 2 rpy=0 0 0 -> xyz=-9 -1 2 rpy=0 0 0

Commit message: running?

File: robot_A.urdf (robot description, URDF)
Before this commit: robot robot, 4 links, 3 joints
Joints:
- joint Torso_BackLeg: origin xyz=-1.5 -1 1 rpy=0 0 0 -> xyz=0.5 -7 1 rpy=0 0 0
- joint Torso_FrontLeg: origin xyz=-0.5 -1 1 rpy=0 0 0 -> xyz=1.5 -7 1 rpy=0 0 0
- joint Torso_Hat: origin xyz=-1 -1 2 rpy=0 0 0 -> xyz=1 -7 2 rpy=0 0 0

File: robot_B.urdf (robot description, URDF)
Before this commit: robot robot, 4 links, 3 joints
Joints:
- joint Torso_BackLeg: origin xyz=-9.5 -1 1 rpy=0 0 0 -> xyz=-7.5 -7 1 rpy=0 0 0
- joint Torso_FrontLeg: origin xyz=-8.5 -1 1 rpy=0 0 0 -> xyz=-6.5 -7 1 rpy=0 0 0
- joint Torso_Hat: origin xyz=-9 -1 2 rpy=0 0 0 -> xyz=-7 -7 2 rpy=0 0 0

Commit message: something is wrong

File: robot_A.urdf (robot description, URDF)
Before this commit: robot robot, 4 links, 3 joints
Joints:
- joint Torso_BackLeg: origin xyz=0.5 -7 1 rpy=0 0 0 -> xyz=-0.5 -1 1 rpy=0 0 0
- joint Torso_FrontLeg: origin xyz=1.5 -7 1 rpy=0 0 0 -> xyz=0.5 -1 1 rpy=0 0 0
- joint Torso_Hat: origin xyz=1 -7 2 rpy=0 0 0 -> xyz=0 -1 2 rpy=0 0 0

File: robot_B.urdf (robot description, URDF)
Before this commit: robot robot, 4 links, 3 joints
Joints:
- joint Torso_BackLeg: origin xyz=-7.5 -7 1 rpy=0 0 0 -> xyz=-6.5 -1 1 rpy=0 0 0
- joint Torso_FrontLeg: origin xyz=-6.5 -7 1 rpy=0 0 0 -> xyz=-5.5 -1 1 rpy=0 0 0
- joint Torso_Hat: origin xyz=-7 -7 2 rpy=0 0 0 -> xyz=-6 -1 2 rpy=0 0 0

Commit message: okay it runs now

File: robot_A.urdf (robot description, URDF)
Before this commit: robot robot, 4 links, 3 joints
Joints:
- joint Torso_BackLeg: origin xyz=-0.5 -1 1 rpy=0 0 0 -> xyz=8.5 -9 1 rpy=0 0 0
- joint Torso_FrontLeg: origin xyz=0.5 -1 1 rpy=0 0 0 -> xyz=9.5 -9 1 rpy=0 0 0
- joint Torso_Hat: origin xyz=0 -1 2 rpy=0 0 0 -> xyz=9 -9 2 rpy=0 0 0

File: robot_B.urdf (robot description, URDF)
Before this commit: robot robot, 4 links, 3 joints
Joints:
- joint Torso_BackLeg: origin xyz=-6.5 -1 1 rpy=0 0 0 -> xyz=-2.5 -9 1 rpy=0 0 0
- joint Torso_FrontLeg: origin xyz=-5.5 -1 1 rpy=0 0 0 -> xyz=-1.5 -9 1 rpy=0 0 0
- joint Torso_Hat: origin xyz=-6 -1 2 rpy=0 0 0 -> xyz=-2 -9 2 rpy=0 0 0

Commit message: it kind of works, I am trying to make there be only one fitness value instead of one for robot A and one for robot B

File: robot_A.urdf (robot description, URDF)
Before this commit: robot robot, 4 links, 3 joints
Joints:
- joint Torso_BackLeg: origin xyz=8.5 -9 1 rpy=0 0 0 -> xyz=3.5 -1 1 rpy=0 0 0
- joint Torso_FrontLeg: origin xyz=9.5 -9 1 rpy=0 0 0 -> xyz=4.5 -1 1 rpy=0 0 0
- joint Torso_Hat: origin xyz=9 -9 2 rpy=0 0 0 -> xyz=4 -1 2 rpy=0 0 0

File: robot_B.urdf (robot description, URDF)
Before this commit: robot robot, 4 links, 3 joints
Joints:
- joint Torso_BackLeg: origin xyz=-2.5 -9 1 rpy=0 0 0 -> xyz=-5.5 -1 1 rpy=0 0 0
- joint Torso_FrontLeg: origin xyz=-1.5 -9 1 rpy=0 0 0 -> xyz=-4.5 -1 1 rpy=0 0 0
- joint Torso_Hat: origin xyz=-2 -9 2 rpy=0 0 0 -> xyz=-5 -1 2 rpy=0 0 0

Commit message: they go towards each other! I had to make it a fitness value for the whole situation, not each robot :)

File: robot_A.urdf (robot description, URDF)
Before this commit: robot robot, 4 links, 3 joints
Joints:
- joint Torso_BackLeg: origin xyz=3.5 -1 1 rpy=0 0 0 -> xyz=1.5 5 1 rpy=0 0 0
- joint Torso_FrontLeg: origin xyz=4.5 -1 1 rpy=0 0 0 -> xyz=2.5 5 1 rpy=0 0 0
- joint Torso_Hat: origin xyz=4 -1 2 rpy=0 0 0 -> xyz=2 5 2 rpy=0 0 0

File: robot_B.urdf (robot description, URDF)
Before this commit: robot robot, 4 links, 3 joints
Joints:
- joint Torso_BackLeg: origin xyz=-5.5 -1 1 rpy=0 0 0 -> xyz=-4.5 5 1 rpy=0 0 0
- joint Torso_FrontLeg: origin xyz=-4.5 -1 1 rpy=0 0 0 -> xyz=-3.5 5 1 rpy=0 0 0
- joint Torso_Hat: origin xyz=-5 -1 2 rpy=0 0 0 -> xyz=-4 5 2 rpy=0 0 0

Commit message: added try except for file opening

File: robot_A.urdf (robot description, URDF)
Before this commit: robot robot, 4 links, 3 joints
Joints:
- joint Torso_BackLeg: origin xyz=1.5 5 1 rpy=0 0 0 -> xyz=-5.5 -4 1 rpy=0 0 0
- joint Torso_FrontLeg: origin xyz=2.5 5 1 rpy=0 0 0 -> xyz=-4.5 -4 1 rpy=0 0 0
- joint Torso_Hat: origin xyz=2 5 2 rpy=0 0 0 -> xyz=-5 -4 2 rpy=0 0 0

File: robot_B.urdf (robot description, URDF)
Before this commit: robot robot, 4 links, 3 joints
Joints:
- joint Torso_BackLeg: origin xyz=-4.5 5 1 rpy=0 0 0 -> xyz=5.5 -4 1 rpy=0 0 0
- joint Torso_FrontLeg: origin xyz=-3.5 5 1 rpy=0 0 0 -> xyz=6.5 -4 1 rpy=0 0 0
- joint Torso_Hat: origin xyz=-4 5 2 rpy=0 0 0 -> xyz=6 -4 2 rpy=0 0 0

Commit message: all is good! nothing broke with the file permissions, I'll test a couple more times

File: robot_A.urdf (robot description, URDF)
Before this commit: robot robot, 4 links, 3 joints
Joints:
- joint Torso_BackLeg: origin xyz=-5.5 -4 1 rpy=0 0 0 -> xyz=2.5 2 1 rpy=0 0 0
- joint Torso_FrontLeg: origin xyz=-4.5 -4 1 rpy=0 0 0 -> xyz=3.5 2 1 rpy=0 0 0
- joint Torso_Hat: origin xyz=-5 -4 2 rpy=0 0 0 -> xyz=3 2 2 rpy=0 0 0

File: robot_B.urdf (robot description, URDF)
Before this commit: robot robot, 4 links, 3 joints
Joints:
- joint Torso_BackLeg: origin xyz=5.5 -4 1 rpy=0 0 0 -> xyz=-3.5 2 1 rpy=0 0 0
- joint Torso_FrontLeg: origin xyz=6.5 -4 1 rpy=0 0 0 -> xyz=-2.5 2 1 rpy=0 0 0
- joint Torso_Hat: origin xyz=6 -4 2 rpy=0 0 0 -> xyz=-3 2 2 rpy=0 0 0

Commit message: got matrix

File: robot_A.urdf (robot description, URDF)
Before this commit: robot robot, 4 links, 3 joints
Links:
- removed link Hat
Joints:
- removed joint Torso_Hat
- joint Torso_BackLeg: origin xyz=2.5 2 1 rpy=0 0 0 -> xyz=-8.5 -6 1 rpy=0 0 0
- joint Torso_FrontLeg: origin xyz=3.5 2 1 rpy=0 0 0 -> xyz=-7.5 -6 1 rpy=0 0 0

File: robot_B.urdf (robot description, URDF)
Before this commit: robot robot, 4 links, 3 joints
Links:
- removed link Hat
Joints:
- removed joint Torso_Hat
- joint Torso_BackLeg: origin xyz=-3.5 2 1 rpy=0 0 0 -> xyz=9.5 -6 1 rpy=0 0 0
- joint Torso_FrontLeg: origin xyz=-2.5 2 1 rpy=0 0 0 -> xyz=10.5 -6 1 rpy=0 0 0

Commit message: matrix writes to csv!

File: robot_A.urdf (robot description, URDF)
Before this commit: robot robot, 3 links, 2 joints
Joints:
- joint Torso_BackLeg: origin xyz=-8.5 -6 1 rpy=0 0 0 -> xyz=-5.5 -4 1 rpy=0 0 0
- joint Torso_FrontLeg: origin xyz=-7.5 -6 1 rpy=0 0 0 -> xyz=-4.5 -4 1 rpy=0 0 0

File: robot_B.urdf (robot description, URDF)
Before this commit: robot robot, 3 links, 2 joints
Joints:
- joint Torso_BackLeg: origin xyz=9.5 -6 1 rpy=0 0 0 -> xyz=6.5 -4 1 rpy=0 0 0
- joint Torso_FrontLeg: origin xyz=10.5 -6 1 rpy=0 0 0 -> xyz=7.5 -4 1 rpy=0 0 0

Commit message: graph works yayayay

File: robot_A.urdf (robot description, URDF)
Before this commit: robot robot, 3 links, 2 joints
Joints:
- joint Torso_BackLeg: origin xyz=-5.5 -4 1 rpy=0 0 0 -> xyz=-0.5 2 1 rpy=0 0 0
- joint Torso_FrontLeg: origin xyz=-4.5 -4 1 rpy=0 0 0 -> xyz=0.5 2 1 rpy=0 0 0

File: robot_B.urdf (robot description, URDF)
Before this commit: robot robot, 3 links, 2 joints
Joints:
- joint Torso_BackLeg: origin xyz=6.5 -4 1 rpy=0 0 0 -> xyz=-10.5 2 1 rpy=0 0 0
- joint Torso_FrontLeg: origin xyz=7.5 -4 1 rpy=0 0 0 -> xyz=-9.5 2 1 rpy=0 0 0
