Commit message: robots working well and the analysis works

File: robot_A.urdf (robot description, URDF)
Before this commit: robot robot, 3 links, 2 joints
Links:
- added link BackLowerLeg, mass 1; collision box size=0.2 0.2 1; visual box size=0.2 0.2 1
- added link FrontLowerLeg, mass 1; collision box size=0.2 0.2 1; visual box size=0.2 0.2 1
- added link LeftLeg, mass 1; collision box size=1 0.2 0.2; visual box size=1 0.2 0.2
- added link LeftLowerLeg, mass 1; collision box size=0.2 0.2 1; visual box size=0.2 0.2 1
- added link RightLeg, mass 1; collision box size=1 0.2 0.2; visual box size=1 0.2 0.2
- added link RightLowerLeg, mass 1; collision box size=0.2 0.2 1; visual box size=0.2 0.2 1
- link BackLeg: geometry collision box size=0.2 1 0.2; visual box size=0.2 1 0.2
- link FrontLeg: geometry collision box size=0.2 1 0.2; visual box size=0.2 1 0.2
Joints:
- added joint BackLeg_BackLowerLeg: type revolute, parent BackLeg, child BackLowerLeg, origin xyz=0 -1 0 rpy=0 0 0, axis 1 0 0, limit lower=-3.14159 upper=3.14159 effort=0.0 velocity=0.0
- added joint FrontLeg_FrontLowerLeg: type revolute, parent FrontLeg, child FrontLowerLeg, origin xyz=0 1 0 rpy=0 0 0, axis 1 0 0, limit lower=-3.14159 upper=3.14159 effort=0.0 velocity=0.0
- added joint LeftLeg_LeftLowerLeg: type revolute, parent LeftLeg, child LeftLowerLeg, origin xyz=-1 0 0 rpy=0 0 0, axis 0 1 0, limit lower=-3.14159 upper=3.14159 effort=0.0 velocity=0.0
- added joint RightLeg_RightLowerLeg: type revolute, parent RightLeg, child RightLowerLeg, origin xyz=1 0 0 rpy=0 0 0, axis 0 1 0, limit lower=-3.14159 upper=3.14159 effort=0.0 velocity=0.0
- added joint Torso_LeftLeg: type revolute, parent Torso, child LeftLeg, origin xyz=-5.5 -9 1 rpy=0 0 0, axis 0 1 0, limit lower=-3.14159 upper=3.14159 effort=0.0 velocity=0.0
- added joint Torso_RightLeg: type revolute, parent Torso, child RightLeg, origin xyz=-4.5 -9 1 rpy=0 0 0, axis 0 1 0, limit lower=-3.14159 upper=3.14159 effort=0.0 velocity=0.0
- joint Torso_BackLeg: axis 0 1 0 -> 1 0 0; origin xyz=-0.5 2 1 rpy=0 0 0 -> xyz=-5 -9.5 1 rpy=0 0 0
- joint Torso_FrontLeg: axis 0 1 0 -> 1 0 0; origin xyz=0.5 2 1 rpy=0 0 0 -> xyz=-5 -8.5 1 rpy=0 0 0

File: robot_B.urdf (robot description, URDF)
Before this commit: robot robot, 3 links, 2 joints
Links:
- added link BackLowerLeg, mass 1; collision box size=0.2 0.2 1; visual box size=0.2 0.2 1
- added link FrontLowerLeg, mass 1; collision box size=0.2 0.2 1; visual box size=0.2 0.2 1
- added link LeftLeg, mass 1; collision box size=1 0.2 0.2; visual box size=1 0.2 0.2
- added link LeftLowerLeg, mass 1; collision box size=0.2 0.2 1; visual box size=0.2 0.2 1
- added link RightLeg, mass 1; collision box size=1 0.2 0.2; visual box size=1 0.2 0.2
- added link RightLowerLeg, mass 1; collision box size=0.2 0.2 1; visual box size=0.2 0.2 1
- link BackLeg: geometry collision box size=0.2 1 0.2; visual box size=0.2 1 0.2
- link FrontLeg: geometry collision box size=0.2 1 0.2; visual box size=0.2 1 0.2
Joints:
- added joint BackLeg_BackLowerLeg: type revolute, parent BackLeg, child BackLowerLeg, origin xyz=0 -1 0 rpy=0 0 0, axis 1 0 0, limit lower=-3.14159 upper=3.14159 effort=0.0 velocity=0.0
- added joint FrontLeg_FrontLowerLeg: type revolute, parent FrontLeg, child FrontLowerLeg, origin xyz=0 1 0 rpy=0 0 0, axis 1 0 0, limit lower=-3.14159 upper=3.14159 effort=0.0 velocity=0.0
- added joint LeftLeg_LeftLowerLeg: type revolute, parent LeftLeg, child LeftLowerLeg, origin xyz=-1 0 0 rpy=0 0 0, axis 0 1 0, limit lower=-3.14159 upper=3.14159 effort=0.0 velocity=0.0
- added joint RightLeg_RightLowerLeg: type revolute, parent RightLeg, child RightLowerLeg, origin xyz=1 0 0 rpy=0 0 0, axis 0 1 0, limit lower=-3.14159 upper=3.14159 effort=0.0 velocity=0.0
- added joint Torso_LeftLeg: type revolute, parent Torso, child LeftLeg, origin xyz=6.5 -9 1 rpy=0 0 0, axis 0 1 0, limit lower=-3.14159 upper=3.14159 effort=0.0 velocity=0.0
- added joint Torso_RightLeg: type revolute, parent Torso, child RightLeg, origin xyz=7.5 -9 1 rpy=0 0 0, axis 0 1 0, limit lower=-3.14159 upper=3.14159 effort=0.0 velocity=0.0
- joint Torso_BackLeg: axis 0 1 0 -> 1 0 0; origin xyz=-10.5 2 1 rpy=0 0 0 -> xyz=7 -9.5 1 rpy=0 0 0
- joint Torso_FrontLeg: axis 0 1 0 -> 1 0 0; origin xyz=-9.5 2 1 rpy=0 0 0 -> xyz=7 -8.5 1 rpy=0 0 0

Commit message: 5 trials of graphs!!

File: robot_A.urdf (robot description, URDF)
Before this commit: robot robot, 9 links, 8 joints
Joints:
- joint Torso_BackLeg: origin xyz=-5 -9.5 1 rpy=0 0 0 -> xyz=0 2.5 1 rpy=0 0 0
- joint Torso_FrontLeg: origin xyz=-5 -8.5 1 rpy=0 0 0 -> xyz=0 3.5 1 rpy=0 0 0
- joint Torso_LeftLeg: origin xyz=-5.5 -9 1 rpy=0 0 0 -> xyz=-0.5 3 1 rpy=0 0 0
- joint Torso_RightLeg: origin xyz=-4.5 -9 1 rpy=0 0 0 -> xyz=0.5 3 1 rpy=0 0 0

File: robot_B.urdf (robot description, URDF)
Before this commit: robot robot, 9 links, 8 joints
Joints:
- joint Torso_BackLeg: origin xyz=7 -9.5 1 rpy=0 0 0 -> xyz=-8 2.5 1 rpy=0 0 0
- joint Torso_FrontLeg: origin xyz=7 -8.5 1 rpy=0 0 0 -> xyz=-8 3.5 1 rpy=0 0 0
- joint Torso_LeftLeg: origin xyz=6.5 -9 1 rpy=0 0 0 -> xyz=-8.5 3 1 rpy=0 0 0
- joint Torso_RightLeg: origin xyz=7.5 -9 1 rpy=0 0 0 -> xyz=-7.5 3 1 rpy=0 0 0

Commit message: working on graphs

File: robot_A.urdf (robot description, URDF)
Before this commit: robot robot, 9 links, 8 joints
Joints:
- joint Torso_BackLeg: origin xyz=0 2.5 1 rpy=0 0 0 -> xyz=-3 2.5 1 rpy=0 0 0
- joint Torso_FrontLeg: origin xyz=0 3.5 1 rpy=0 0 0 -> xyz=-3 3.5 1 rpy=0 0 0
- joint Torso_LeftLeg: origin xyz=-0.5 3 1 rpy=0 0 0 -> xyz=-3.5 3 1 rpy=0 0 0
- joint Torso_RightLeg: origin xyz=0.5 3 1 rpy=0 0 0 -> xyz=-2.5 3 1 rpy=0 0 0

File: robot_B.urdf (robot description, URDF)
Before this commit: robot robot, 9 links, 8 joints
Joints:
- joint Torso_BackLeg: origin xyz=-8 2.5 1 rpy=0 0 0 -> xyz=7 2.5 1 rpy=0 0 0
- joint Torso_FrontLeg: origin xyz=-8 3.5 1 rpy=0 0 0 -> xyz=7 3.5 1 rpy=0 0 0
- joint Torso_LeftLeg: origin xyz=-8.5 3 1 rpy=0 0 0 -> xyz=6.5 3 1 rpy=0 0 0
- joint Torso_RightLeg: origin xyz=-7.5 3 1 rpy=0 0 0 -> xyz=7.5 3 1 rpy=0 0 0

Commit message: more trials!!!

File: robot_A.urdf (robot description, URDF)
Before this commit: robot robot, 9 links, 8 joints
Joints:
- joint Torso_BackLeg: origin xyz=-3 2.5 1 rpy=0 0 0 -> xyz=3 -4.5 1 rpy=0 0 0
- joint Torso_FrontLeg: origin xyz=-3 3.5 1 rpy=0 0 0 -> xyz=3 -3.5 1 rpy=0 0 0
- joint Torso_LeftLeg: origin xyz=-3.5 3 1 rpy=0 0 0 -> xyz=2.5 -4 1 rpy=0 0 0
- joint Torso_RightLeg: origin xyz=-2.5 3 1 rpy=0 0 0 -> xyz=3.5 -4 1 rpy=0 0 0

File: robot_B.urdf (robot description, URDF)
Before this commit: robot robot, 9 links, 8 joints
Joints:
- joint Torso_BackLeg: origin xyz=7 2.5 1 rpy=0 0 0 -> xyz=-6 -4.5 1 rpy=0 0 0
- joint Torso_FrontLeg: origin xyz=7 3.5 1 rpy=0 0 0 -> xyz=-6 -3.5 1 rpy=0 0 0
- joint Torso_LeftLeg: origin xyz=6.5 3 1 rpy=0 0 0 -> xyz=-6.5 -4 1 rpy=0 0 0
- joint Torso_RightLeg: origin xyz=7.5 3 1 rpy=0 0 0 -> xyz=-5.5 -4 1 rpy=0 0 0

Commit message: 50 trials! done with data collection!

File: robot_A.urdf (robot description, URDF)
Before this commit: robot robot, 9 links, 8 joints
Joints:
- joint Torso_BackLeg: origin xyz=3 -4.5 1 rpy=0 0 0 -> xyz=0 2.5 1 rpy=0 0 0
- joint Torso_FrontLeg: origin xyz=3 -3.5 1 rpy=0 0 0 -> xyz=0 3.5 1 rpy=0 0 0
- joint Torso_LeftLeg: origin xyz=2.5 -4 1 rpy=0 0 0 -> xyz=-0.5 3 1 rpy=0 0 0
- joint Torso_RightLeg: origin xyz=3.5 -4 1 rpy=0 0 0 -> xyz=0.5 3 1 rpy=0 0 0

File: robot_B.urdf (robot description, URDF)
Before this commit: robot robot, 9 links, 8 joints
Joints:
- joint Torso_BackLeg: origin xyz=-6 -4.5 1 rpy=0 0 0 -> xyz=-8 2.5 1 rpy=0 0 0
- joint Torso_FrontLeg: origin xyz=-6 -3.5 1 rpy=0 0 0 -> xyz=-8 3.5 1 rpy=0 0 0
- joint Torso_LeftLeg: origin xyz=-6.5 -4 1 rpy=0 0 0 -> xyz=-8.5 3 1 rpy=0 0 0
- joint Torso_RightLeg: origin xyz=-5.5 -4 1 rpy=0 0 0 -> xyz=-7.5 3 1 rpy=0 0 0
